File: StmRelay.kicad_pcb (KiCad board)
At the start: 4 copper layers, 36 x 48 mm, 8 parts, among them J2 Conn_02x10_Odd_Even, U1 TXS0108EPW, U2 TXS0108EPW

Commit message: last modifs before shipping
Parts:
- C1, C2, C3, C4: footprint Capacitor_SMD:C_0201_0603Metric -> Capacitor_SMD:C_0603_1608Metric_Pad1.08x0.95mm_HandSolder
Routing:
- net +5V: track 74.8 -> 79.1 mm
- net GND: track 13.5 -> 13.0 mm
